Commit message: robot spawned in gazebogazebo

File: src/krever/urdf/krever.urdf (robot description, URDF)
Before this commit: robot krever, 12 links, 11 joints
Links:
- link caster_wheel1: geometry collision sphere radius=0.05; visual sphere radius=0.05
- link caster_wheel2: geometry collision sphere radius=0.05; visual sphere radius=0.05
Joints:
- removed joint base_left_wheel_joint
- removed joint base_right_wheel_joint
- added joint left_wheel_joint: type continuous, parent base_link, child left_wheel, origin xyz=0 0.315 0.05 rpy=0 0 0, axis 0 1 0, limit effort=10.0 velocity=5.0
- added joint right_wheel_joint: type continuous, parent base_link, child right_wheel, origin xyz=-0 -0.315 0.05 rpy=0 0 0, axis 0 1 0, limit effort=10.0 velocity=5.0

Commit message: testing teleop on rasp4

File: src/krever/urdf/krever.urdf (robot description, URDF)
Before this commit: robot krever, 12 links, 11 joints
Links:
- link caster_wheel1: geometry collision sphere radius=0.045; visual sphere radius=0.045
- link caster_wheel2: geometry collision sphere radius=0.045; visual sphere radius=0.045
Joints:
- joint base_suppot_joint: origin xyz=-0.265 0. 0.76 rpy=0.0 0.0 0.0 -> xyz=-0.255 0. 0.725 rpy=0.0 0.0 0.0
- joint center_rod_joint: origin xyz=0 0 0.555 rpy=0.0 0.0 1.57 -> xyz=0 0 0.52 rpy=0.0 0.0 1.57
- joint left_rod_joint: origin xyz=0.25 0.25 0.555 rpy=0.0 0.0 0 -> xyz=0.25 0.25 0.52 rpy=0.0 0.0 0
- joint right_rod_joint: origin xyz=0.25 -0.25 0.555 rpy=0.0 0.0 0 -> xyz=0.25 -0.25 0.52 rpy=0.0 0.0 0
- joint tray_joint: origin xyz=0.27 0.0 -0.465 rpy=0.0 0.0 0.0 -> xyz=0.27 0.0 -0.43 rpy=0.0 0.0 0.0
